File: HW2/ME433/ME433_songwei.sch (EAGLE design)
At the start: 22 parts, among them J1 USB-MB-H

Commit message: Worked on .brd and edited .sch
Parts:
- removed R5, R6: 10k, ME433_songwei:R-US_0207/12
- added R3, R4: 10k, resistor:R-US_0207/10
Connections:
- net +3V3: now also R3.2, R4.2; no longer R5.2, R6.2
- net B4/USER: now also R3.1; no longer R5.1
- net MCLR: now also R4.1; no longer R6.1
Changed lines of the file:
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@@
 <part name="+3V7" library="ME433_songwei" deviceset="+3V3" device=""/>
 <part name="+3V8" library="ME433_songwei" deviceset="+3V3" device=""/>
-<part name="R5" library="ME433_songwei" deviceset="R-US_" device="0207/12" value="10k"/>
-<part name="R6" library="ME433_songwei" deviceset="R-US_" device="0207/12" value="10k"/>
 <part name="GND20" library="ME433_songwei" deviceset="GND" device=""/>
 <part name="GND21" library="ME433_songwei" deviceset="GND" device=""/>
 <part name="P+3" library="ME433_songwei" deviceset="+5V" device=""/>
 <part name="+3V9" library="ME433_songwei" deviceset="+3V3" device=""/>
+<part name="R3" library="resistor" deviceset="R-US_" device="0207/10" value="10k"/>
+<part name="R4" library="resistor" deviceset="R-US_" device="0207/10" value="10k"/>
 </parts>
 <sheets>
@@
 <instance part="+3V7" gate="G$1" x="101.6" y="30.48"/>
 <instance part="+3V8" gate="G$1" x="86.36" y="17.78"/>
-<instance part="R5" gate="G$1" x="86.36" y="5.08" rot="R90"/>
-<instance part="R6" gate="G$1" x="101.6" y="20.32" rot="R90"/>
 <instance part="GND20" gate="1" x="121.92" y="7.62"/>
 <instance part="GND21" gate="1" x="106.68" y="-17.78"/>
 <instance part="P+3" gate="1" x="162.56" y="17.78"/>
 <instance part="+3V9" gate="G$1" x="162.56" y="-12.7"/>
+<instance part="R3" gate="G$1" x="86.36" y="5.08" rot="R90"/>
+<instance part="R4" gate="G$1" x="101.6" y="20.32" rot="R90"/>
 </instances>
 <busses>
@@
 <segment>
 <pinref part="+3V8" gate="G$1" pin="+3V3"/>
-<pinref part="R5" gate="G$1" pin="2"/>
 <wire x1="86.36" y1="15.24" x2="86.36" y2="10.16" width="0.1524" layer="91"/>
-</segment>
-<segment>
-<pinref part="R6" gate="G$1" pin="2"/>
+<pinref part="R3" gate="G$1" pin="2"/>
+</segment>
+<segment>
 <pinref part="+3V7" gate="G$1" pin="+3V3"/>
 <wire x1="101.6" y1="25.4" x2="101.6" y2="27.94" width="0.1524" layer="91"/>
+<pinref part="R4" gate="G$1" pin="2"/>
 </segment>
 <segment>
@@
 <segment>
 <pinref part="U$4" gate="G$1" pin="1"/>
-<pinref part="R6" gate="G$1" pin="1"/>
 <wire x1="101.6" y1="12.7" x2="101.6" y2="15.24" width="0.1524" layer="91"/>
 <wire x1="101.6" y1="12.7" x2="93.98" y2="12.7" width="0.1524" layer="91"/>
 <junction x="101.6" y="12.7"/>
 <label x="93.98" y="12.7" size="1.778" layer="95"/>
+<pinref part="R4" gate="G$1" pin="1"/>
 </segment>
 </net>
@@
 </segment>
 <segment>
-<pinref part="R5" gate="G$1" pin="1"/>
 <pinref part="U$5" gate="G$1" pin="1"/>
 <wire x1="86.36" y1="0" x2="86.36" y2="-10.16" width="0.1524" layer="91"/>
@@
 <junction x="86.36" y="-10.16"/>
 <label x="76.2" y="-10.16" size="1.778" layer="95"/>
-</segment>
-<segment>
+<pinref part="R3" gate="G$1" pin="1"/>
+</segment>
+<segment>
